File: hardware/Business Card v2.kicad_sch (KiCad schematic)
At the start: 39 parts, among them J1 Conn_01x03_Pin, Q1 DMP21D0UFB4-P, U1 ATTINY816-MNR, U3 NT3H2111W0FHKH

Commit message: 調布組込みラボ版 NFC 基板名刺
WiHarper/nfc_card（752793d）のフォーク。シルクを調布組込みラボ版に差し替え、
JLCPCB で部品実装まで発注できるよう BOM を修正した（C1 の LCSC 番号の
サイズ違いを修正、R4 に LCSC 番号を追加、JLCPCB 用の製造データを追加）。
回路・アンテナ・部品配置・配線は元の設計のまま。変更点は docs/CHANGES.md に記録。

Co-Authored-By: Claude Opus 5.5 <noreply@anthropic.com>
Parts:
- C1: LCSC C1639 -> C1552
- R4: LCSC (none) -> C25076
Changed lines of the file:
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@@
+			)
+		)
+		(property "LCSC" "C25076"
+			(at 29.21 128.778 90)
+			(effects
+				(font
+					(size 1.27 1.27)
+				)
+				(hide yes)
 			)
 		)
@@
 			)
 		)
-		(property "LCSC" "C1639"
+		(property "LCSC" "C1552"
 			(at 49.53 49.53 0)
 			(effects
